Commit message: Actividad 2 final: Pipeline UDP, Exploración reactiva LIDAR con SensorData QoS, y fix crítico de PyAudio Segmentation Fault en microfono

File: src/project_bringup/urdf/turtlebot3_waffle_pi_custom.urdf (robot description, URDF)
Before this commit: robot turtlebot3_waffle_pi, 11 links, 10 joints
Joints:
- joint ${namespace}scan_joint: origin xyz=-0.064 0.1 0.122 rpy=0 0 0 -> xyz=-0.064 -0.05 0.122 rpy=0 0 0
